File: GCEW_Glove/GCEW_Glove.sch (KiCad schematic (older format))
At the start: 9 parts, among them U1 TLV809-DBV, U2 LM3668, U3 ATMEGA328PB-AU, U4 HC-05_BluetoothModule

Commit message: GCEW Glove Schematic Update 1
Parts:
- added C2, C5, C6, C7: 0.1uF 25V, symbol C
- added J1: Flex_Sensor_Inputs, symbol Conn_01x06
- added J2: Programmer, symbol Conn_01x06
- added R1, R2, R3: R, symbol R
- added SW1: SW_SPDT, symbol SW_SPDT
- added SW2: SW_Push, symbol SW_Push
- C4: renamed from C2; value 22uF 16V -> 22uF 25V
Connections:
- net +3V3: now also C6.2, C7.2, J1.1 (Pin_1), J1.3 (Pin_3), J1.5 (Pin_5), J2.1 (Pin_1)
- net GND: now also C2.1, C5.2, C6.1, C7.1, J2.6 (Pin_6), R1.2, R2.2, R3.2, SW1.2 (B), SW2.2; no longer BT1.2 (GND)
- net VCC: now also C2.2
- net MOSI: now reaches U3.15 ((MOSI0/TXD1/OC2A/PTCXY)PB3)
- net MOSI: now also J2.2 (Pin_2)
- net MISO: now reaches U3.16 ((MISO0/RXD1/PTCXY)PB4)
- net MISO: now also J2.3 (Pin_3)
- net SCK: now reaches U3.17 ((XCK1/SCK0/PTCXY)PB5)
- net SCK: now also J2.4 (Pin_4)
- net at U3.20 (AREF): now also C5.1
- net Flex_1: now reaches U3.25 ((ADC2/PTCY)PC2)
- net Flex_1: now also J1.2 (Pin_2), R1.1
- net Flex_2: now reaches U3.26 ((ADC3/PTCY)PC3)
- net Flex_2: now also J1.4 (Pin_4), R2.1
- net Flex_3: now reaches U3.27 ((SDA0/ADC4/PTCY)PC4)
- net Flex_3: now also J1.6 (Pin_6), R3.1
- net ~RESET: now reaches U3.29 ((~RESET~)PC6)
- net ~RESET: now also J2.5 (Pin_5)
- net at U3.9 ((OC0B/T1/PTCXY)PD5): now also SW2.1
- new net: BT1.2 (GND), SW1.1 (A)
- no-connect marks 17 -> 18
Other:
- moved on the sheet: C3

Commit message: GCEW Glove Schematic Update 2
Parts:
- added D1, D2: LED_ARGB, symbol LED_ARGB
- added R1, R2, R3, R4, R5, R6: R, symbol R
- renumbered J2 to J1, J1 to J2, R1 to R7, R2 to R8, R3 to R9
Connections:
- net +3V3: now also D1.1 (A), D2.1 (A)
- net at U3.10 ((OC0A/AIN0/PTCXY)PD6): now also R6.2
- net at U3.11 ((AIN1/PTCXY)PD7): now also SW2.1
- net at U3.19 (PE2(PTCY/ADC6/ICP3/~SS1~)): now also R3.1
- net at U3.2 ((XCK0/T0/PTCXY)PD4): now also R4.2; no longer U4.6 (EN)
- net at U3.23 ((MISO1/ADC0/PTCY)PC0): now also U4.6 (EN)
- net at U3.3 (PE0(PTCXY/SDA1/ICP4/ACO)): now also R1.1
- net at U3.6 (PE1(PTCXY/SCL1/T4)): now also R2.1
- net at U3.9 ((OC0B/T1/PTCXY)PD5): now also R5.2; no longer SW2.1
- new net: D1.2 (RK), R3.2
- new net: D1.3 (GK), R2.2
- new net: D1.4 (BK), R1.2
- new net: D2.2 (RK), R4.1
- new net: D2.3 (GK), R5.1
- new net: D2.4 (BK), R6.1
- no-connect marks 18 -> 12
Other:
- moved on the sheet: J2, R7, R8, R9, SW2
