File: schematic is dramatic/GCEW/GCEW.sch (KiCad schematic (older format))
At the start: 38 parts, among them J1 Conn_01x09_Male, Q1 Q_NMOS_DGS, Q2 Q_NMOS_DGS, Q3 Q_NMOS_DGS, Q4 Q_NMOS_DGS, Q5 Q_NMOS_DGS, Q6 Q_NMOS_DGS, U1 DRV8323RHRGZ, U2 BLDCMOTOR, U3 LM26CIM5-VHA

Commit message: GCEW Motor Controller Schematic Update 1
Parts:
- removed C10: 15uF, 25TQC15MYFB:CAPPM3528X200N, symbol Device:C
- removed C11: 100nF, Capacitor_SMD:C_1206_3216Metric, symbol Device:C
- removed Q1, Q2, Q3, Q4, Q5, Q6: Q_NMOS_DGS, Package_TO_SOT_SMD:TO-263-2, symbol myLib:IPB029N06N
- removed R10: 10.4k, Resistor_SMD:R_0805_2012Metric, symbol Device:R
- removed R11: 57.6k, Resistor_SMD:R_0402_1005Metric, symbol Device:R
- removed R12, R13, R14: 2m, Resistor_SMD:R_1206_3216Metric, symbol Device:R
- removed R9: 100k, Resistor_SMD:R_1206_3216Metric, symbol Device:R
- removed U1: DRV8323RHRGZ, myLib:TI-RGZ-QFN-48-1EP_7x7mm_Pitch0.5mm, symbol symbols:DRV8323RHRGZ
- removed U2: BLDCMOTOR, TerminalBlock:TerminalBlock_Altech_AK300-3_P5.00mm, symbol symbols:BLDCMOTOR
- removed VDC1: 36V, TerminalBlock:TerminalBlock_Altech_AK300-3_P5.00mm, symbol Device:Battery
- added BT1: Battery, symbol myLib:Battery
- added M1: BLDC_Motor, symbol myLib:BLDC_Motor
- added U2: DRV8323RH, myLib:TI-RGZ-QFN-48-1EP_7x7mm_Pitch0.5mm, symbol myLib:DRV8323RH
- added U3, U4, U5, U6, U7, U8: IPB029N06N, symbol myLib:IPB029N06N
- added U9: BLDC_Hall_Sensor, symbol myLib:BLDC_Hall_Sensor
- C2: value 1uF -> 100nF; footprint Capacitor_SMD:C_1206_3216Metric -> (none)
- C3: value 47nF -> 10nF; footprint Capacitor_SMD:C_1206_3216Metric -> (none)
- C4: value 100nF -> 10nF; footprint Capacitor_SMD:C_1206_3216Metric -> (none)
- C5, C8: footprint Capacitor_SMD:C_1206_3216Metric -> (none)
- C6: value 10nF -> 47nF; footprint Capacitor_SMD:C_1206_3216Metric -> (none)
- C7: value 10nF -> 1uF; footprint Capacitor_SMD:C_1206_3216Metric -> (none)
- C9: value 4.7uF -> 15uF; footprint CAPAE430X550N:CAPAE430X550N -> (none)
- L1: value 220uH -> L; footprint CLF10060NIT-1R0N-D:INDPM101100X630N -> (none)
- R1, R2, R3: value 10k -> R; footprint Resistor_SMD:R_1206_3216Metric -> (none)
- R4: value 1M -> 57.6K; footprint Resistor_SMD:R_1206_3216Metric -> (none)
- R5: value 18k -> 10.4K; footprint Resistor_SMD:R_1206_3216Metric -> (none)
- R6: value 18k -> 2milli; footprint Resistor_SMD:R_1206_3216Metric -> (none)
- R7: value 1M -> 2milli; footprint Resistor_SMD:R_1206_3216Metric -> (none)
- R8: value 100k -> 2milli; footprint Resistor_SMD:R_1206_3216Metric -> (none)
- renumbered U3 to U1
Connections:
- net labels added: +5V, 36V, DVDD, GHA, GHB, GHC, GLA, GLB, GLC, Hall_A, Hall_B, Hall_C, Over_Temp, SNA, SNB, SNC, SPA, SPB, SPC
- net labels removed: +BATT, 5V, 5v, H_A, H_B, H_C, VCC, Vtemp
- wire segments 156 -> 101
- no-connect marks 3 -> 1
Other:
- moved on the sheet: C1, D1, J1, U1

Commit message: GCEW Motor Controller Schematic Update 2
Parts:
- added C8: 4.7uF 80V, symbol Device:C
- added R4: 100K, symbol Device:R
- renumbered C9 to C10, C8 to C9, R4 to R5, R5 to R6, R6 to R7, R7 to R8, R8 to R9
Connections:
- net 36V: now also C8.1, R4.2
- net GND: now also C8.2
- net at U2.48 (nSHDN): now also R4.1
Changed lines of the file:
@@
 EESchema Schematic File Version 4
-LIBS:GCEW-cache
 EELAYER 26 0
 EELAYER END
@@
 $EndComp
 $Comp
-L power:GND #PWR02
+L power:GND #PWR01
 U 1 1 5BC834DF
 P 1000 1450
-F 0 "#PWR02" H 1000 1200 50  0001 C CNN
+F 0 "#PWR01" H 1000 1200 50  0001 C CNN
 F 1 "GND" H 1005 1277 50  0000 C CNN
 F 2 "" H 1000 1450 50  0001 C CNN
@@
 SOC
 $Comp
-L power:GND #PWR07
+L power:GND #PWR06
 U 1 1 5BD16A03
 P 1500 6400
-F 0 "#PWR07" H 1500 6150 50  0001 C CNN
+F 0 "#PWR06" H 1500 6150 50  0001 C CNN
 F 1 "GND" H 1505 6227 50  0000 C CNN
 F 2 "" H 1500 6400 50  0001 C CNN
@@
 $EndComp
 $Comp
-L power:GND #PWR05
+L power:GND #PWR02
 U 1 1 5BD17970
 P 1000 5950
-F 0 "#PWR05" H 1000 5700 50  0001 C CNN
+F 0 "#PWR02" H 1000 5700 50  0001 C CNN
 F 1 "GND" V 1005 5822 50  0000 R CNN
 F 2 "" H 1000 5950 50  0001 C CNN
@@
 	4450 3300 4350 3300
 $Comp
-L Device:C C8
+L Device:C C9
 U 1 1 5BDA1890
 P 7800 4700
-F 0 "C8" H 7915 4746 50  0000 L CNN
+F 0 "C9" H 7915 4746 50  0000 L CNN
 F 1 "100nF" H 7915 4655 50  0000 L CNN
 F 2 "" H 7838 4550 50  0001 C CNN
@@
 	4450 1900 4150 1900
 $Comp
-L power:GNDA #PWR013
+L power:GNDA #PWR011
 U 1 1 5BDA2FAD
 P 5500 5250
-F 0 "#PWR013" H 5500 5000 50  0001 C CNN
+F 0 "#PWR011" H 5500 5000 50  0001 C CNN
 F 1 "GNDA" H 5505 5077 50  0000 C CNN
 F 2 "" H 5500 5250 50  0001 C CNN
@@
 	5500 5250 5500 5050
 $Comp
-L power:GND #PWR014
+L power:GND #PWR012
 U 1 1 5BDA32CC
 P 5750 5250
-F 0 "#PWR014" H 5750 5000 50  0001 C CNN
+F 0 "#PWR012" H 5750 5000 50  0001 C CNN
 F 1 "GND" H 5755 5077 50  0000 C CNN
 F 2 "" H 5750 5250 50  0001 C CNN
@@
 $EndComp
 $Comp
-L power:GND #PWR011
+L power:GND #PWR010
 U 1 1 5BDA3307
 P 5200 5250
-F 0 "#PWR011" H 5200 5000 50  0001 C CNN
+F 0 "#PWR010" H 5200 5000 50  0001 C CNN
 F 1 "GND" H 5205 5077 50  0000 C CNN
 F 2 "" H 5200 5250 50  0001 C CNN
@@
 SOA
 $Comp
-L power:+5V #PWR06
+L power:+5V #PWR05
 U 1 1 5BDA560E
 P 1500 5350
-F 0 "#PWR06" H 1500 5200 50  0001 C CNN
+F 0 "#PWR05" H 1500 5200 50  0001 C CNN
 F 1 "+5V" H 1515 5523 50  0000 C CNN
 F 2 "" H 1500 5350 50  0001 C CNN
@@
 $EndComp
 $Comp
-L power:+5V #PWR017
+L power:+5V #PWR016
 U 1 1 5BDA56B5
 P 8800 5200
-F 0 "#PWR017" H 8800 5050 50  0001 C CNN
+F 0 "#PWR016" H 8800 5050 50  0001 C CNN
 F 1 "+5V" H 8815 5373 50  0000 C CNN
 F 2 "" H 8800 5200 50  0001 C CNN
@@
 $EndComp
 $Comp
-L Device:R R4
+L Device:R R5
 U 1 1 5BDA5775
 P 7800 5400
-F 0 "R4" H 7870 5446 50  0000 L CNN
+F 0 "R5" H 7870 5446 50  0000 L CNN
 F 1 "57.6K" H 7870 5355 50  0000 L CNN
 F 2 "" V 7730 5400 50  0001 C CNN
@@
 $EndComp
 $Comp
-L Device:R R5
+L Device:R R6
 U 1 1 5BDA57C9
 P 7800 5800
-F 0 "R5" H 7870 5846 50  0000 L CNN
+F 0 "R6" H 7870 5846 50  0000 L CNN
 F 1 "10.4K" H 7870 5755 50  0000 L CNN
 F 2 "" V 7730 5800 50  0001 C CNN
@@
 	6900 4750 6650 4750
 $Comp
-L power:GND #PWR015
+L power:GND #PWR014
 U 1 1 5BDA6FAD
 P 7800 6050
-F 0 "#PWR015" H 7800 5800 50  0001 C CNN
+F 0 "#PWR014" H 7800 5800 50  0001 C CNN
 F 1 "GND" H 7805 5877 50  0000 C CNN
 F 2 "" H 7800 6050 50  0001 C CNN
@@
 $EndComp
 $Comp
-L Device:C C9
+L Device:C C10
 U 1 1 5BDA7581
 P 8350 5350
-F 0 "C9" H 8465 5396 50  0000 L CNN
+F 0 "C10" H 8465 5396 50  0000 L CNN
 F 1 "15uF" H 8465 5305 50  0000 L CNN
 F 2 "" H 8388 5200 50  0001 C CNN
@@
 Hall_C
 $Comp
-L power:GND #PWR022
+L power:GND #PWR020
 U 1 1 5BDAD196
 P 12550 3200
-F 0 "#PWR022" H 12550 2950 50  0001 C CNN
+F 0 "#PWR020" H 12550 2950 50  0001 C CNN
 F 1 "GND" H 12555 3027 50  0000 C CNN
 F 2 "" H 12550 3200 50  0001 C CNN
@@
 $EndComp
 $Comp
-L power:+5V #PWR021
+L power:+5V #PWR019
 U 1 1 5BDAD1EB
 P 12550 2800
-F 0 "#PWR021" H 12550 2650 50  0001 C CNN
+F 0 "#PWR019" H 12550 2650 50  0001 C CNN
 F 1 "+5V" H 12565 2973 50  0000 C CNN
 F 2 "" H 12550 2800 50  0001 C CNN
@@
 SNA
 $Comp
-L Device:R R6
+L Device:R R7
 U 1 1 5BDC0FC0
 P 7950 3900
-F 0 "R6" H 8020 3946 50  0000 L CNN
+F 0 "R7" H 8020 3946 50  0000 L CNN
 F 1 "2milli" H 8020 3855 50  0000 L CNN
 F 2 "" V 7880 3900 50  0001 C CNN
@@
 $EndComp
 $Comp
-L power:GND #PWR016
+L power:GND #PWR015
 U 1 1 5BDC102D
 P 7950 4050
-F 0 "#PWR016" H 7950 3800 50  0001 C CNN
+F 0 "#PWR015" H 7950 3800 50  0001 C CNN
 F 1 "GND" H 7955 3877 50  0000 C CNN
 F 2 "" H 7950 4050 50  0001 C CNN
@@
 SNA
 $Comp
-L Device:R R7
+L Device:R R8
 U 1 1 5BDC2200
 P 9050 3900
-F 0 "R7" H 9120 3946 50  0000 L CNN
+F 0 "R8" H 9120 3946 50  0000 L CNN
 F 1 "2milli" H 9120 3855 50  0000 L CNN
 F 2 "" V 8980 3900 50  0001 C CNN
@@
 $EndComp
 $Comp
-L Device:R R8
+L Device:R R9
 U 1 1 5BDC226A
 P 10150 3900
-F 0 "R8" H 10220 3946 50  0000 L CNN
+F 0 "R9" H 10220 3946 50  0000 L CNN
 F 1 "2milli" H 10220 3855 50  0000 L CNN
 F 2 "" V 10080 3900 50  0001 C CNN
@@
 $EndComp
 $Comp
-L power:GND #PWR019
+L power:GND #PWR017
 U 1 1 5BDC23F0
 P 9050 4050
-F 0 "#PWR019" H 9050 3800 50  0001 C CNN
+F 0 "#PWR017" H 9050 3800 50  0001 C CNN
 F 1 "GND" H 9055 3877 50  0000 C CNN
 F 2 "" H 9050 4050 50  0001 C CNN
@@
 $EndComp
 $Comp
-L power:GND #PWR020
+L power:GND #PWR018
 U 1 1 5BDC242B
 P 10150 4050
-F 0 "#PWR020" H 10150 3800 50  0001 C CNN
+F 0 "#PWR018" H 10150 3800 50  0001 C CNN
 F 1 "GND" H 10155 3877 50  0000 C CNN
 F 2 "" H 10150 4050 50  0001 C CNN
@@
 	3750 3900 3750 3650
 $Comp
-L power:GND #PWR010
+L power:GND #PWR09
 U 1 1 5BE040E2
 P 3400 4450
-F 0 "#PWR010" H 3400 4200 50  0001 C CNN
+F 0 "#PWR09" H 3400 4200 50  0001 C CNN
 F 1 "GND" H 3405 4277 50  0000 C CNN
 F 2 "" H 3400 4450 50  0001 C CNN
@@
 	5400 1200 5400 1250
 $Comp
-L power:PWR_FLAG #FLG0101
+L power:PWR_FLAG #FLG01
 U 1 1 5BE18940
 P 2200 800
-F 0 "#FLG0101" H 2200 875 50  0001 C CNN
+F 0 "#FLG01" H 2200 875 50  0001 C CNN
 F 1 "PWR_FLAG" H 2100 1000 50  0000 C CNN
 F 2 "" H 2200 800 50  0001 C CNN
@@
 $EndComp
 $Comp
-L power:+5V #PWR0101
+L power:+5V #PWR07
 U 1 1 5BE18946
 P 2400 800
-F 0 "#PWR0101" H 2400 650 50  0001 C CNN
+F 0 "#PWR07" H 2400 650 50  0001 C CNN
 F 1 "+5V" H 2450 1000 50  0000 C CNN
 F 2 "" H 2400 800 50  0001 C CNN
@@
 	2400 800  2200 800
 $Comp
-L power:PWR_FLAG #FLG0102
+L power:PWR_FLAG #FLG02
 U 1 1 5BE266D4
 P 2950 800
-F 0 "#FLG0102" H 2950 875 50  0001 C CNN
+F 0 "#FLG02" H 2950 875 50  0001 C CNN
 F 1 "PWR_FLAG" H 2950 974 50  0000 C CNN
 F 2 "" H 2950 800 50  0001 C CNN
@@
 $EndComp
 $Comp
-L power:GNDA #PWR0102
+L power:GNDA #PWR08
 U 1 1 5BE2678E
 P 2950 850
-F 0 "#PWR0102" H 2950 600 50  0001 C CNN
+F 0 "#PWR08" H 2950 600 50  0001 C CNN
 F 1 "GNDA" H 2955 677 50  0000 C CNN
 F 2 "" H 2950 850 50  0001 C CNN
@@
 	5800 1250 5500 1250
 Connection ~ 5500 1250
+$Comp
+L Device:C C8
+U 1 1 5BD0BC2B
+P 6000 1450
+F 0 "C8" H 6115 1496 50  0000 L CNN
+F 1 "4.7uF 80V" H 6115 1405 50  0000 L CNN
+F 2 "" H 6038 1300 50  0001 C CNN
+F 3 "~" H 6000 1450 50  0001 C CNN
+	1    6000 1450
+	1    0    0    -1
+$EndComp
+Wire Wire Line
+	6000 1300 6000 1250
+Wire Wire Line
+	6000 1250 5800 1250
+Connection ~ 5800 1250
+$Comp
+L power:GND #PWR013
+U 1 1 5BD121CF
+P 6000 1650
+F 0 "#PWR013" H 6000 1400 50  0001 C CNN
+F 1 "GND" H 6005 1477 50  0000 C CNN
+F 2 "" H 6000 1650 50  0001 C CNN
+F 3 "" H 6000 1650 50  0001 C CNN
+	1    6000 1650
+	1    0    0    -1
+$EndComp
+Wire Wire Line
+	6000 1650 6000 1600
+$Comp
+L Device:R R4
+U 1 1 5BD1581A
+P 4250 4550
+F 0 "R4" V 4043 4550 50  0000 C CNN
+F 1 "100K" V 4134 4550 50  0000 C CNN
+F 2 "" V 4180 4550 50  0001 C CNN
+F 3 "~" H 4250 4550 50  0001 C CNN
+	1    4250 4550
+	0    1    1    0
+$EndComp
+Wire Wire Line
+	4400 4550 4450 4550
+Text GLabel 4100 4550 0    50   Input ~ 0
+VIN
+Text GLabel 5800 1250 1    50   Input ~ 0
+VIN
 $EndSCHEMATC

Commit message: GCEW Motor Controller Schematic Update 3
Parts:
- added C12: 0.1uF 25V, symbol Device:C
- added C2: 1uF 50V, symbol Device:C
- added C8: 33uF 100V, symbol Device:C
- added C9: 0.1uF 100V, symbol Device:C
- added J2, J3: Conn_02x03_Odd_Even, symbol Connector_Generic:Conn_02x03_Odd_Even
- added J4: Conn_02x02_Odd_Even, symbol Connector_Generic:Conn_02x02_Odd_Even
- added R1, R11: 10K, symbol Device:R
- added R10: 47K, symbol Device:R
- added R13, R5, R9: 1M, symbol Device:R
- added R3, R7: 18K, symbol Device:R
- added R4, R6: 75K, symbol Device:R
- C10: renamed from C7; value 1uF -> 1uF 50V
- C13: renamed from C9; value 100nF -> 0.1uF 25V
- C14: renamed from C10; value 15uF -> 15uF 25V
- J1: symbol Connector:Conn_01x09_Male -> Connector:Conn_01x10_Female
- L1: value L -> 220uH
- renumbered C8 to C11, C2 to C3, C3 to C4, C4 to C5, C5 to C6, C6 to C7, R3 to R12, R4 to R14, R5 to R15, R6 to R16, R7 to R17, R8 to R18, R9 to R19, R1 to R2, R2 to R8
Connections:
- net +5V: now also J1.2 (Pin_2), U2.26 (VREF), C12.1, R1.1; no longer J1.8 (Pin_8)
- net 36V: now also C8.1, C9.1
- net CAL: now also J1.7 (Pin_7); no longer J1.4 (Pin_4)
- net DVDD: now also C2.1, R11.1, R3.2, R4.2
- net GND: now also D1.2 (A), J1.1 (Pin_1), C2.2, C8.2, C9.2; no longer J1.9 (Pin_9)
- net GNDA: now also C12.2, J3.5 (Pin_5), R10.2, R13.2, R5.2, R6.2, R7.2, R9.2
- net INHA: now also J1.10 (Pin_10); no longer J1.1 (Pin_1)
- net INHC: now also J1.9 (Pin_9); no longer J1.2 (Pin_2)
- net INLC: now also J1.8 (Pin_8); no longer J1.3 (Pin_3)
- net SOA: now also J1.4 (Pin_4); no longer J1.7 (Pin_7)
- net SOB: now also J1.5 (Pin_5); no longer J1.6 (Pin_6)
- net SOC: now also J1.6 (Pin_6); no longer J1.5 (Pin_5)
- net at C13.2, D1.1 (K), L1.1: now also U2.45 (SW)
- net at U2.28 (nFault): now also R11.2
- net at U2.29 (MODE): now also R13.1
- net IDRIVE: now reaches U2.30 (IDRIVE)
- net IDRIVE: now also J2.2 (Pin_2), J2.4 (Pin_4), J2.6 (Pin_6)
- net VDS: now reaches U2.31 (VDS)
- net VDS: now also J3.2 (Pin_2), J3.4 (Pin_4), J3.6 (Pin_6)
- net GAIN: now reaches U2.32 (GAIN)
- net GAIN: now also J4.2 (Pin_2), J4.4 (Pin_4)
- net Over_Temp renamed ENABLE
- net ENABLE: now also J1.3 (Pin_3), R1.2
- new net: J4.1 (Pin_1), R9.1
- new net: J4.3 (Pin_3), R10.1
- new net: J3.1 (Pin_1), R6.1
- new net: J3.3 (Pin_3), R7.1
- new net: J2.1 (Pin_1), R3.1
- new net: J2.3 (Pin_3), R4.1
- new net: J2.5 (Pin_5), R5.1
Other:
- moved on the sheet: C11, D1

Commit message: GCEW Motor Controller Schematic Update 4
Parts:
- C10, C12, C13, C2, C3, C4, C5, C6, C7, C9: footprint (none) -> Capacitor_SMD:C_1206_3216Metric
- C11: footprint (none) -> CAPAE430X550N:CAPAE430X550N
- C14: footprint (none) -> 25TQC15MYFB:CAPPM3528X200N
- C8: footprint (none) -> Capacitor_THT:CP_Radial_D10.0mm_P5.00mm
- L1: footprint (none) -> CLF10060NIT-1R0N-D:INDPM101100X630N
- R1, R10, R11, R12, R13, R14, R17, R18, R19, R2, R3, R4, R5, R6, R7, R8, R9: footprint (none) -> Resistor_SMD:R_1206_3216Metric
- R15, R16: footprint (none) -> Resistor_SMD:R_0805_2012Metric
- U3, U4, U5, U6, U7, U8: footprint (none) -> Package_TO_SOT_SMD:TO-263-2
Changed lines of the file:
@@
 F 0 "C13" H 7915 4746 50  0000 L CNN
 F 1 "0.1uF 25V" H 7915 4655 50  0000 L CNN
-F 2 "" H 7838 4550 50  0001 C CNN
+F 2 "Capacitor_SMD:C_1206_3216Metric" H 7838 4550 50  0001 C CNN
 F 3 "~" H 7800 4700 50  0001 C CNN
 	1    7800 4700
@@
 F 0 "C10" H 5550 1500 50  0000 R CNN
 F 1 "1uF 50V" H 5700 1600 50  0000 R CNN
-F 2 "" H 5338 1350 50  0001 C CNN
+F 2 "Capacitor_SMD:C_1206_3216Metric" H 5338 1350 50  0001 C CNN
 F 3 "~" H 5300 1500 50  0001 C CNN
 	1    5300 1500
@@
 F 0 "C7" H 3900 2100 50  0000 L CNN
 F 1 "47nF" H 3900 1950 50  0000 L CNN
-F 2 "" H 4188 1900 50  0001 C CNN
+F 2 "Capacitor_SMD:C_1206_3216Metric" H 4188 1900 50  0001 C CNN
 F 3 "~" H 4150 2050 50  0001 C CNN
 	1    4150 2050
@@
 F 0 "R15" H 7870 5446 50  0000 L CNN
 F 1 "57.6K" H 7870 5355 50  0000 L CNN
-F 2 "" V 7730 5400 50  0001 C CNN
+F 2 "Resistor_SMD:R_0805_2012Metric" V 7730 5400 50  0001 C CNN
 F 3 "~" H 7800 5400 50  0001 C CNN
 	1    7800 5400
@@
 F 0 "R16" H 7870 5846 50  0000 L CNN
 F 1 "10.4K" H 7870 5755 50  0000 L CNN
-F 2 "" V 7730 5800 50  0001 C CNN
+F 2 "Resistor_SMD:R_0805_2012Metric" V 7730 5800 50  0001 C CNN
 F 3 "~" H 7800 5800 50  0001 C CNN
 	1    7800 5800
@@
 F 0 "C14" H 8465 5396 50  0000 L CNN
 F 1 "15uF 25V" H 8465 5305 50  0000 L CNN
-F 2 "" H 8388 5200 50  0001 C CNN
+F 2 "25TQC15MYFB:CAPPM3528X200N" H 8388 5200 50  0001 C CNN
 F 3 "~" H 8350 5350 50  0001 C CNN
 	1    8350 5350
@@
 F 0 "L1" H 7853 5046 50  0000 L CNN
 F 1 "220uH" H 7853 4955 50  0000 L CNN
-F 2 "" H 7800 5000 50  0001 C CNN
+F 2 "CLF10060NIT-1R0N-D:INDPM101100X630N" H 7800 5000 50  0001 C CNN
 F 3 "~" H 7800 5000 50  0001 C CNN
 	1    7800 5000
@@
 F 0 "U3" H 8130 2396 50  0000 L CNN
 F 1 "IPB029N06N" H 8050 2550 50  0000 L CNN
-F 2 "" H 7950 2350 50  0001 C CNN
+F 2 "Package_TO_SOT_SMD:TO-263-2" H 7950 2350 50  0001 C CNN
 F 3 "" H 7950 2350 50  0001 C CNN
 	1    7950 2350
@@
 F 0 "U5" H 9230 2396 50  0000 L CNN
 F 1 "IPB029N06N" H 9150 2550 50  0000 L CNN
-F 2 "" H 9050 2350 50  0001 C CNN
+F 2 "Package_TO_SOT_SMD:TO-263-2" H 9050 2350 50  0001 C CNN
 F 3 "" H 9050 2350 50  0001 C CNN
 	1    9050 2350
@@
 F 0 "U7" H 10330 2396 50  0000 L CNN
 F 1 "IPB029N06N" H 10250 2550 50  0000 L CNN
-F 2 "" H 10150 2350 50  0001 C CNN
+F 2 "Package_TO_SOT_SMD:TO-263-2" H 10150 2350 50  0001 C CNN
 F 3 "" H 10150 2350 50  0001 C CNN
 	1    10150 2350
@@
 F 0 "U4" H 8130 3546 50  0000 L CNN
 F 1 "IPB029N06N" H 8050 3700 50  0000 L CNN
-F 2 "" H 7950 3500 50  0001 C CNN
+F 2 "Package_TO_SOT_SMD:TO-263-2" H 7950 3500 50  0001 C CNN
 F 3 "" H 7950 3500 50  0001 C CNN
 	1    7950 3500
@@
 F 0 "U6" H 9230 3546 50  0000 L CNN
 F 1 "IPB029N06N" H 9150 3700 50  0000 L CNN
-F 2 "" H 9050 3500 50  0001 C CNN
+F 2 "Package_TO_SOT_SMD:TO-263-2" H 9050 3500 50  0001 C CNN
 F 3 "" H 9050 3500 50  0001 C CNN
 	1    9050 3500
@@
 F 0 "U8" H 10330 3546 50  0000 L CNN
 F 1 "IPB029N06N" H 10250 3700 50  0000 L CNN
-F 2 "" H 10150 3500 50  0001 C CNN
+F 2 "Package_TO_SOT_SMD:TO-263-2" H 10150 3500 50  0001 C CNN
 F 3 "" H 10150 3500 50  0001 C CNN
 	1    10150 3500
@@
 F 0 "R17" H 8020 3946 50  0000 L CNN
 F 1 "2milli" H 8020 3855 50  0000 L CNN
-F 2 "" V 7880 3900 50  0001 C CNN
+F 2 "Resistor_SMD:R_1206_3216Metric" V 7880 3900 50  0001 C CNN
 F 3 "~" H 7950 3900 50  0001 C CNN
 	1    7950 3900
@@
 F 0 "R18" H 9120 3946 50  0000 L CNN
 F 1 "2milli" H 9120 3855 50  0000 L CNN
-F 2 "" V 8980 3900 50  0001 C CNN
+F 2 "Resistor_SMD:R_1206_3216Metric" V 8980 3900 50  0001 C CNN
 F 3 "~" H 9050 3900 50  0001 C CNN
 	1    9050 3900
@@
 F 0 "R19" H 10220 3946 50  0000 L CNN
 F 1 "2milli" H 10220 3855 50  0000 L CNN
-F 2 "" V 10080 3900 50  0001 C CNN
+F 2 "Resistor_SMD:R_1206_3216Metric" V 10080 3900 50  0001 C CNN
 F 3 "~" H 10150 3900 50  0001 C CNN
 	1    10150 3900
@@
 F 0 "R12" H 3820 3546 50  0000 L CNN
 F 1 "R" H 3820 3455 50  0000 L CNN
-F 2 "" V 3680 3500 50  0001 C CNN
+F 2 "Resistor_SMD:R_1206_3216Metric" V 3680 3500 50  0001 C CNN
 F 3 "~" H 3750 3500 50  0001 C CNN
 	1    3750 3500
@@
 F 0 "C6" H 3865 4196 50  0000 L CNN
 F 1 "10nF" H 3900 4050 50  0000 L CNN
-F 2 "" H 3788 4000 50  0001 C CNN
+F 2 "Capacitor_SMD:C_1206_3216Metric" H 3788 4000 50  0001 C CNN
 F 3 "~" H 3750 4150 50  0001 C CNN
 	1    3750 4150
@@
 F 0 "R8" H 3470 3546 50  0000 L CNN
 F 1 "R" H 3470 3455 50  0000 L CNN
-F 2 "" V 3330 3500 50  0001 C CNN
+F 2 "Resistor_SMD:R_1206_3216Metric" V 3330 3500 50  0001 C CNN
 F 3 "~" H 3400 3500 50  0001 C CNN
 	1    3400 3500
@@
 F 0 "R2" H 3120 3546 50  0000 L CNN
 F 1 "R" H 3120 3455 50  0000 L CNN
-F 2 "" V 2980 3500 50  0001 C CNN
+F 2 "Resistor_SMD:R_1206_3216Metric" V 2980 3500 50  0001 C CNN
 F 3 "~" H 3050 3500 50  0001 C CNN
 	1    3050 3500
@@
 F 0 "C5" H 3515 4196 50  0000 L CNN
 F 1 "10nF" H 3500 4050 50  0000 L CNN
-F 2 "" H 3438 4000 50  0001 C CNN
+F 2 "Capacitor_SMD:C_1206_3216Metric" H 3438 4000 50  0001 C CNN
 F 3 "~" H 3400 4150 50  0001 C CNN
 	1    3400 4150
@@
 F 0 "C4" H 3165 4196 50  0000 L CNN
 F 1 "10nF" H 3150 4050 50  0000 L CNN
-F 2 "" H 3088 4000 50  0001 C CNN
+F 2 "Capacitor_SMD:C_1206_3216Metric" H 3088 4000 50  0001 C CNN
 F 3 "~" H 3050 4150 50  0001 C CNN
 	1    3050 4150
@@
 F 0 "C3" H 2050 3800 50  0000 L CNN
 F 1 "100nF" H 2000 3700 50  0000 L CNN
-F 2 "" H 2338 3650 50  0001 C CNN
+F 2 "Capacitor_SMD:C_1206_3216Metric" H 2338 3650 50  0001 C CNN
 F 3 "~" H 2300 3800 50  0001 C CNN
 	1    2300 3800
@@
 F 0 "C11" H 6215 1446 50  0000 L CNN
 F 1 "4.7uF 80V" H 6215 1355 50  0000 L CNN
-F 2 "" H 6138 1250 50  0001 C CNN
+F 2 "CAPAE430X550N:CAPAE430X550N" H 6138 1250 50  0001 C CNN
 F 3 "~" H 6100 1400 50  0001 C CNN
 	1    6100 1400
@@
 F 0 "R14" V 4043 4550 50  0000 C CNN
 F 1 "100K" V 4134 4550 50  0000 C CNN
-F 2 "" V 4180 4550 50  0001 C CNN
+F 2 "Resistor_SMD:R_1206_3216Metric" V 4180 4550 50  0001 C CNN
 F 3 "~" H 4250 4550 50  0001 C CNN
 	1    4250 4550
@@
 F 0 "R11" V 3957 2600 50  0000 C CNN
 F 1 "10K" V 3866 2600 50  0000 C CNN
-F 2 "" V 3680 2600 50  0001 C CNN
+F 2 "Resistor_SMD:R_1206_3216Metric" V 3680 2600 50  0001 C CNN
 F 3 "~" H 3750 2600 50  0001 C CNN
 	1    3750 2600
@@
 F 0 "R13" V 4100 2650 50  0000 C CNN
 F 1 "1M" V 4100 2800 50  0000 C CNN
-F 2 "" V 4130 2800 50  0001 C CNN
+F 2 "Resistor_SMD:R_1206_3216Metric" V 4130 2800 50  0001 C CNN
 F 3 "~" H 4200 2800 50  0001 C CNN
 	1    4200 2800
@@
 F 0 "R3" V 3250 5250 50  0000 C CNN
 F 1 "18K" V 3250 5450 50  0000 C CNN
-F 2 "" V 3280 5300 50  0001 C CNN
+F 2 "Resistor_SMD:R_1206_3216Metric" V 3280 5300 50  0001 C CNN
 F 3 "~" H 3350 5300 50  0001 C CNN
 	1    3350 5300
@@
 F 0 "R4" V 3250 5450 50  0000 C CNN
 F 1 "75K" V 3250 5650 50  0000 C CNN
-F 2 "" V 3280 5500 50  0001 C CNN
+F 2 "Resistor_SMD:R_1206_3216Metric" V 3280 5500 50  0001 C CNN
 F 3 "~" H 3350 5500 50  0001 C CNN
 	1    3350 5500
@@
 F 0 "R6" V 3250 6050 50  0000 C CNN
 F 1 "75K" V 3250 6250 50  0000 C CNN
-F 2 "" V 3280 6100 50  0001 C CNN
+F 2 "Resistor_SMD:R_1206_3216Metric" V 3280 6100 50  0001 C CNN
 F 3 "~" H 3350 6100 50  0001 C CNN
 	1    3350 6100
@@
 F 0 "R7" V 3250 6250 50  0000 C CNN
 F 1 "18K" V 3250 6450 50  0000 C CNN
-F 2 "" V 3280 6300 50  0001 C CNN
+F 2 "Resistor_SMD:R_1206_3216Metric" V 3280 6300 50  0001 C CNN
 F 3 "~" H 3350 6300 50  0001 C CNN
 	1    3350 6300
@@
 F 0 "R5" V 3250 5650 50  0000 C CNN
 F 1 "1M" V 3250 5850 50  0000 C CNN
-F 2 "" V 3280 5700 50  0001 C CNN
+F 2 "Resistor_SMD:R_1206_3216Metric" V 3280 5700 50  0001 C CNN
 F 3 "~" H 3350 5700 50  0001 C CNN
 	1    3350 5700
@@
 F 0 "R9" V 3300 6800 50  0000 C CNN
 F 1 "1M" V 3300 7000 50  0000 C CNN
-F 2 "" V 3330 6850 50  0001 C CNN
+F 2 "Resistor_SMD:R_1206_3216Metric" V 3330 6850 50  0001 C CNN
 F 3 "~" H 3400 6850 50  0001 C CNN
 	1    3400 6850
@@
 F 0 "R10" V 3300 7000 50  0000 C CNN
 F 1 "47K" V 3300 7200 50  0000 C CNN
-F 2 "" V 3330 7050 50  0001 C CNN
+F 2 "Resistor_SMD:R_1206_3216Metric" V 3330 7050 50  0001 C CNN
 F 3 "~" H 3400 7050 50  0001 C CNN
 	1    3400 7050
@@
 F 0 "C12" H 6965 1446 50  0000 L CNN
 F 1 "0.1uF 25V" H 6965 1355 50  0000 L CNN
-F 2 "" H 6888 1250 50  0001 C CNN
+F 2 "Capacitor_SMD:C_1206_3216Metric" H 6888 1250 50  0001 C CNN
 F 3 "~" H 6850 1400 50  0001 C CNN
 	1    6850 1400
@@
 F 0 "R1" H 2370 5796 50  0000 L CNN
 F 1 "10K" H 2370 5705 50  0000 L CNN
-F 2 "" V 2230 5750 50  0001 C CNN
+F 2 "Resistor_SMD:R_1206_3216Metric" V 2230 5750 50  0001 C CNN
 F 3 "~" H 2300 5750 50  0001 C CNN
 	1    2300 5750
@@
 F 0 "C2" H 1600 3800 50  0000 L CNN
 F 1 "1uF 50V" H 1450 3700 50  0000 L CNN
-F 2 "" H 1888 3650 50  0001 C CNN
+F 2 "Capacitor_SMD:C_1206_3216Metric" H 1888 3650 50  0001 C CNN
 F 3 "~" H 1850 3800 50  0001 C CNN
 	1    1850 3800
@@
 F 0 "C9" V 4550 1200 50  0000 C CNN
 F 1 "0.1uF 100V" V 4550 1500 50  0000 C CNN
-F 2 "" H 4738 1250 50  0001 C CNN
+F 2 "Capacitor_SMD:C_1206_3216Metric" H 4738 1250 50  0001 C CNN
 F 3 "~" H 4700 1400 50  0001 C CNN
 	1    4700 1400
@@
 F 0 "C8" V 4550 900 50  0000 C CNN
 F 1 "33uF 100V" V 4550 1200 50  0000 C CNN
-F 2 "" H 4738 950 50  0001 C CNN
+F 2 "Capacitor_THT:CP_Radial_D10.0mm_P5.00mm" H 4738 950 50  0001 C CNN
 F 3 "~" H 4700 1100 50  0001 C CNN
 	1    4700 1100
