File: GCEW Motor Controller MCU/GCEW Motor Controller MCU.kicad_pcb (KiCad board)
At the start: 2 copper layers, 54 x 48 mm, 9 parts, among them J1 POWER IN, J2 MC2, J3 MC1, J4 Programmer, U1 ATmega328PB-AU, U2 HC-05_BluetoothModule

Commit message: GCEW Motor Controller MCU PCB Update 2
Finalized GCEW Motor Controller MCU PCB. Added bottom silkscreen text for input connectors. Generated gerber files for manufacturer.
Other:
- board text added: "+5V"
- board text added: "CAL2"
- board text added: "EN2"
- board text added: "INHA2"
- board text added: "INLC2"
- board text added: "SOB2"
- board text added: "SOC2"
Changed lines of the file:
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@@
   (general
     (thickness 1.6)
-    (drawings 25)
+    (drawings 35)
     (tracks 190)
     (zones 0)
@@
   (layers
     (0 F.Cu signal)
-    (31 B.Cu signal hide)
+    (31 B.Cu signal)
     (32 B.Adhes user)
     (33 F.Adhes user)
@@
   )
   (setup
-    (last_trace_width 0.3)
+    (last_trace_width 0.25)
     (user_trace_width 0.2)
     (user_trace_width 0.25)
@@
     (user_trace_width 0.5)
     (trace_clearance 0.2)
-    (zone_clearance 0.4)
+    (zone_clearance 0.5)
     (zone_45_only no)
     (trace_min 0.2)
@@
     (pcbplotparams
       (layerselection 0x010fc_ffffffff)
-      (usegerberextensions false)
+      (usegerberextensions true)
       (usegerberattributes false)
       (usegerberadvancedattributes false)
@@
       (psa4output false)
       (plotreference true)
-      (plotvalue true)
+      (plotvalue false)
       (plotinvisibletext false)
       (padsonsilk false)
@@
       (outputformat 1)
       (mirror false)
-      (drillshape 1)
+      (drillshape 0)
       (scaleselection 1)
-      (outputdirectory ""))
+      (outputdirectory "GCEW Motor Controller MCU Gerbers/"))
   )
   (net 0 "")
@@
     (pad 1 thru_hole circle (at -11.5 1.3) (size 2.5 2.5) (drill 1.25) (layers *.Cu *.Mask)
       (net 2 INHC1))
+  )
+  (gr_text GND (at 141 93.5 270) (layer B.SilkS)
+    (effects (font (size 1 1) (thickness 0.2)) (justify mirror))
+  )
+  (gr_text +5V (at 141.25 89.25 270) (layer B.SilkS)
+    (effects (font (size 1 1) (thickness 0.2)) (justify mirror))
+  )
+  (gr_text INHC1 (at 156 70.5 180) (layer B.SilkS)
+    (effects (font (size 1 1) (thickness 0.2)) (justify mirror))
+  )
+  (gr_text INLC2 (at 159.5 68.85 180) (layer B.SilkS)
+    (effects (font (size 1 1) (thickness 0.2)) (justify mirror))
+  )
+  (gr_text EN2 (at 166.5 68.95 180) (layer B.SilkS)
+    (effects (font (size 1 1) (thickness 0.2)) (justify mirror))
+  )
+  (gr_text CAL2 (at 163 70.5 180) (layer B.SilkS)
+    (effects (font (size 1 1) (thickness 0.2)) (justify mirror))
+  )
+  (gr_text INHA2 (at 152.5 68.9 180) (layer B.SilkS)
+    (effects (font (size 1 1) (thickness 0.2)) (justify mirror))
+  )
+  (gr_text SOC2 (at 177 70.5 180) (layer B.SilkS)
+    (effects (font (size 1 1) (thickness 0.2)) (justify mirror))
+  )
+  (gr_text SOB2 (at 173.5 68.9 180) (layer B.SilkS)
+    (effects (font (size 1 1) (thickness 0.2)) (justify mirror))
+  )
+  (gr_text SOA1 (at 170.075 70.5 180) (layer B.SilkS)
+    (effects (font (size 1 1) (thickness 0.2)) (justify mirror))
   )
   (gr_text MOSI (at 149.25 98.85 270) (layer B.SilkS)
@@
   (segment (start 174.75 93) (end 173.95 93) (width 0.3) (layer F.Cu) (net 27))
   (zone (net 17) (net_name GND) (layer B.Cu) (hatch edge 0.508)
-    (connect_pads (clearance 0.4))
+    (connect_pads (clearance 0.5))
     (min_thickness 0.254)
     (fill yes (arc_segments 16) (thermal_gap 0.508) (thermal_bridge_width 1))
