File: GCEW Motor Controller MCU KiCAD/GCEW Motor Controller MCU.kicad_pcb (KiCad board)
At the start: 2 copper layers, 54 x 48 mm, 9 parts, among them J1 POWER IN, J2 MC2, J3 MC1, J4 Programmer, U1 ATmega328PB-AU, U2 HC-05_BluetoothModule

Commit message: Reorganized Files
Other:
- board text added: "SOA2"
Changed lines of the file:
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@@
   (layers
     (0 F.Cu signal)
-    (31 B.Cu signal)
+    (31 B.Cu signal hide)
     (32 B.Adhes user)
     (33 F.Adhes user)
@@
     (pcbplotparams
       (layerselection 0x010fc_ffffffff)
-      (usegerberextensions false)
+      (usegerberextensions true)
       (usegerberattributes false)
       (usegerberadvancedattributes false)
@@
       (psa4output false)
       (plotreference true)
-      (plotvalue true)
+      (plotvalue false)
       (plotinvisibletext false)
       (padsonsilk false)
@@
       (outputformat 1)
       (mirror false)
-      (drillshape 1)
+      (drillshape 0)
       (scaleselection 1)
-      (outputdirectory ""))
+      (outputdirectory "GCEW Motor Controller MCU Gerbers/"))
   )
   (net 0 "")
@@
     (pad 1 thru_hole circle (at -1 1.3 270) (size 2.5 2.5) (drill 1.25) (layers *.Cu *.Mask)
       (net 18 +5V))
+    (model ${KISYS3DMOD}/Terminal_Blocks.3dshapes/TerminalBlock_Pheonix_PT-3.5mm_2pol.wrl
+      (offset (xyz -1 -1.25 0))
+      (scale (xyz 1 1 1))
+      (rotate (xyz 0 0 0))
+    )
   )
   (module myLib:PhoenixContact_1985027_8-Pin-Connector_8A_P3.5mm (layer F.Cu)
@@
     (pad 8 thru_hole circle (at 13 1.3 180) (size 2.5 2.5) (drill 1.25) (layers *.Cu *.Mask)
       (net 16 INHA2))
+    (model ${KISYS3DMOD}/Terminal_Blocks.3dshapes/TerminalBlock_Pheonix_PT-3.5mm_8pol.wrl
+      (offset (xyz -11.5 -1.25 0))
+      (scale (xyz 1 1 1))
+      (rotate (xyz 0 0 0))
+    )
   )
   (module myLib:PhoenixContact_1985027_8-Pin-Connector_8A_P3.5mm (layer F.Cu)
@@
     (pad 1 thru_hole circle (at -11.5 1.3) (size 2.5 2.5) (drill 1.25) (layers *.Cu *.Mask)
       (net 2 INHC1))
+    (model ${KISYS3DMOD}/Terminal_Blocks.3dshapes/TerminalBlock_Pheonix_PT-3.5mm_8pol.wrl
+      (offset (xyz -11.5 -1.25 0))
+      (scale (xyz 1 1 1))
+      (rotate (xyz 0 0 0))
+    )
   )
   (gr_text GND (at 141 93.5 270) (layer B.SilkS)
@@
     (effects (font (size 1 1) (thickness 0.2)) (justify mirror))
   )
-  (gr_text SOA1 (at 170.075 70.5 180) (layer B.SilkS)
-    (effects (font (size 1 1) (thickness 0.2)) (justify mirror))
-  )
+  (gr_text SOA2 (at 170.075 70.5 180) (layer B.SilkS)
+    (effects (font (size 1 1) (thickness 0.2)) (justify mirror))
+  )
